File: telinksensor-hw.kicad_sch (KiCad schematic)
At the start: 81 parts, among them J1 ANT, J2 3W RTD, J4 RTD 2W, J5 SOIC bite, Q1 2N7002, SW1 SW_Push, U1 TLSR8258, U2 SHT40, U3 BMP390, Y1 24MHz

Commit message: Routing done
Parts:
- removed J1: ANT, Connector_Coaxial:U.FL_Molex_MCRF_73412-0110_Vertical, symbol Connector:Conn_Coaxial
- removed R8: 0R, Resistor_SMD:R_0402_1005Metric, symbol Device:R
- removed TP1: PGA+, TestPoint:TestPoint_Pad_D1.0mm, symbol Connector:TestPoint
- removed TP3: PGA-, TestPoint:TestPoint_Pad_D1.0mm, symbol Connector:TestPoint
- added BT1: CR2032-BS-6-1, Battery:BatteryHolder_Keystone_1060_1x2032, symbol Device:Battery_Cell
- added TP11: MM8130-2600, murrata:MM8130-2600, symbol Connector:CoaxialSwitch_Testpoint
- gave numbers to parts that had none: 1
Connections:
- net GND: now also BT1.2 (-), TP11.G
- net VDD: now also BT1.1 (+)
- net at R10.2, R17.1: now also J2.1 (Pin_1); no longer J2.3 (Pin_3)
- net at C20.1, L3.2: now also TP11.C; no longer C18.1
- net at R13.1, R15.2: now also J2.3 (Pin_3); no longer J2.1 (Pin_1)
- new net: C18.1, TP11.A
Other:
- moved on the sheet: AE1, C17, C18
